File: Assets/Design Blocks/Shrimps.kicad_blocks/Shrimp - Arduino Mega.kicad_block/Shrimp - Arduino Mega.kicad_sch (KiCad schematic)
At the start: 1 part

Commit message: Added Arduino stuff
Parts:
- renumbered XA1 to XA?
Connections:
- net +5V: now reaches XA?.5V1 (5V)
- net +5V: now also XA?.5V3 (5V), XA?.5V4 (5V)
- net GND: now reaches XA?.GND1 (GND)
- net GND: now also XA?.GND2 (GND), XA?.GND3 (GND), XA?.GND5 (GND), XA?.GND6 (GND)
